Commit message: completed upper body

File: gk_description/urdf/arms/left_arm.urdf.xacro (robot description, xacro)
@@ -51,5 +51,5 @@
             </inertial>
         <visual>
-            <origin xyz="0 0 -0.042" rpy="0 0 0"/>
+            <origin xyz="0 0 -0.042" rpy="0 0 ${PI}"/>
             <geometry>
                 <mesh filename="package://gk_description/meshes/STL/ARMS/left_arm.stl" />
@@ -58,5 +58,5 @@
         </visual>
         <collision>
-            <origin xyz="0 0 -0.042" rpy="0 0 0"/>
+            <origin xyz="0 0 -0.042" rpy="0 0 ${PI}"/>
             <geometry>
                 <mesh filename="package://gk_description/meshes/STL/ARMS/left_arm.stl" />

File: gk_description/urdf/arms/right_arm.urdf.xacro (robot description, xacro)
@@ -51,5 +51,5 @@
             </inertial>
         <visual>
-            <origin xyz="0 0 -0.042" rpy="0 0 0"/>
+            <origin xyz="0 0 -0.042" rpy="0 0 ${PI}"/>
             <geometry>
                 <mesh filename="package://gk_description/meshes/STL/ARMS/right_arm.stl" />
@@ -58,5 +58,5 @@
         </visual>
         <collision>
-            <origin xyz="0 0 -0.042" rpy="0 0 0"/>
+            <origin xyz="0 0 -0.042" rpy="0 0 ${PI}"/>
             <geometry>
                 <mesh filename="package://gk_description/meshes/STL/ARMS/right_arm.stl" />
