Commit message: added height

File: gk_description/urdf/body/body.urdf.xacro (robot description, xacro)
@@ -5,5 +5,5 @@
         <parent link="base_link" />
         <child link="body_link" />
-        <origin xyz="-0.005 0 0" rpy="0 0 0"/>
+        <origin xyz="-0.005 0 0.4" rpy="0 0 0"/>
     </joint>
     <!-- base body -->

Commit message: change frame

File: gk_description/urdf/body/body.urdf.xacro (robot description, xacro)
@@ -5,5 +5,5 @@
         <parent link="base_link" />
         <child link="body_link" />
-        <origin xyz="-0.005 0 0.4" rpy="0 0 0"/>
+        <origin xyz="-0.005 0 0.0" rpy="0 0 0"/>
     </joint>
     <!-- base body -->
