Commit message: added gazebo plugin and effort transmission

File: gk_description/robots/ganken_kun_v1.xacro (robot description, xacro)
@@ -18,5 +18,15 @@
     <xacro:include filename="$(find gk_description)/urdf/arms/right_arm.urdf.xacro"/>
     <xacro:include filename="$(find gk_description)/urdf/head/head.urdf.xacro"/>
+    <xacro:include filename="$(find gk_description)/urdf/legs/right_leg.urdf.xacro"/>
     <xacro:include filename="$(find gk_description)/urdf/legs/left_leg.urdf.xacro"/>
-    <xacro:include filename="$(find gk_description)/urdf/legs/right_leg.urdf.xacro"/>
+    <!-- Import transmission -->
+    <xacro:include filename="$(find gk_description)/urdf/arms/arm.transmission.xacro" />
+    <xacro:include filename="$(find gk_description)/urdf/head/head.transmission.xacro" />
+    <xacro:include filename="$(find gk_description)/urdf/legs/leg.transmission.xacro" />
+    <!-- Import gazebo plugin -->
+    <xacro:include filename="$(find gk_description)/urdf/gazebo.xacro"/>
+    <xacro:include filename="$(find gk_description)/urdf/body/body.gazebo.xacro"/>
+    <xacro:include filename="$(find gk_description)/urdf/arms/arm.gazebo.xacro" />
+    <xacro:include filename="$(find gk_description)/urdf/head/head.gazebo.xacro" />
+    <xacro:include filename="$(find gk_description)/urdf/legs/leg.gazebo.xacro" />
 </robot>

File: gk_description/urdf/arms/left_arm.urdf.xacro (robot description, xacro)
@@ -6,5 +6,5 @@
         <child link="left_body_to_arm_link" />
         <origin xyz="0 0.07 0.1" rpy="0 0 0" />
-        <limit effort="1000" lower="${-PI}" upper="${PI}" velocity="1.0" />
+        <limit effort="1000" lower="${-3*PI/4}" upper="${3*PI/4}" velocity="1.0" />
         <axis xyz="0 1 0" />
     </joint>
@@ -20,5 +20,5 @@
         <child link="left_hand_link" />
         <origin xyz="0 0 -0.084" rpy="0 ${PI/2} 0" />
-        <limit effort="1000" lower="${-PI}" upper="${PI}" velocity="1.0" />
+        <limit effort="1000" lower="${-3*PI/4}" upper="${3*PI/4}" velocity="1.0" />
         <axis xyz="0 1 0" />
     </joint>

File: gk_description/urdf/arms/right_arm.urdf.xacro (robot description, xacro)
@@ -6,5 +6,5 @@
         <child link="right_body_to_arm_link" />
         <origin xyz="0 -0.07 0.1" rpy="0 0 0" />
-        <limit effort="1000" lower="${-PI}" upper="${PI}" velocity="1.0" />
+        <limit effort="1000" lower="${-3*PI/4}" upper="${3*PI/4}" velocity="1.0" />
         <axis xyz="0 1 0" />
     </joint>
@@ -20,5 +20,5 @@
         <child link="right_hand_link" />
         <origin xyz="0 0 -0.084" rpy="0 ${PI/2} 0" />
-        <limit effort="1000" lower="${-PI}" upper="${PI}" velocity="1.0" />
+        <limit effort="1000" lower="${-3*PI/4}" upper="${3*PI/4}" velocity="1.0" />
         <axis xyz="0 1 0" />
     </joint>

File: gk_description/urdf/head/head.urdf.xacro (robot description, xacro)
@@ -6,5 +6,5 @@
         <child link="head_yaw_link" />
         <origin xyz="0 0 0.152" rpy="0 0 0" />
-        <limit effort="1000" lower="${-PI}" upper="${PI}" velocity="1.0" />
+        <limit effort="1000" lower="${-3*PI/4}" upper="${3*PI/4}" velocity="1.0" />
         <axis xyz="0 0 1" />
     </joint>

File: gk_description/urdf/legs/left_leg.urdf.xacro (robot description, xacro)
@@ -6,5 +6,5 @@
         <child link="left_waist_yaw_link" />
         <origin xyz="0.005 0.044 -0.0575" rpy="0 0 0" />
-        <limit effort="1000" lower="${-PI}" upper="${PI}" velocity="1.0" />
+        <limit effort="1000" lower="${-3*PI/4}" upper="${3*PI/4}" velocity="1.0" />
         <axis xyz="0 0 1" />
     </joint>
@@ -66,5 +66,5 @@
         <child link="left_ankle_pitch_link" />
         <origin xyz="0 0 0" rpy="0 0 0" />
-        <limit effort="1000" lower="${-PI}" upper="${PI}" velocity="1.0" />
+        <limit effort="1000" lower="${-3*PI/4}" upper="${3*PI/4}" velocity="1.0" />
         <axis xyz="0 1 0" />
     </joint>

File: gk_description/urdf/legs/right_leg.urdf.xacro (robot description, xacro)
@@ -6,5 +6,5 @@
         <child link="right_waist_yaw_link" />
         <origin xyz="0.005 -0.044 -0.0575" rpy="0 0 0" />
-        <limit effort="1000" lower="${-PI}" upper="${PI}" velocity="1.0" />
+        <limit effort="1000" lower="${-3*PI/4}" upper="${3*PI/4}" velocity="1.0" />
         <axis xyz="0 0 1" />
     </joint>
@@ -66,5 +66,5 @@
         <child link="right_ankle_pitch_link" />
         <origin xyz="0 0 0" rpy="0 0 0" />
-        <limit effort="1000" lower="${-PI}" upper="${PI}" velocity="1.0" />
+        <limit effort="1000" lower="${-3*PI/4}" upper="${3*PI/4}" velocity="1.0" />
         <axis xyz="0 1 0" />
     </joint>

Commit message: fix bug

File: gk_description/robots/ganken_kun_v1.xacro (robot description, xacro)
@@ -6,6 +6,7 @@
     <xacro:include filename="$(find gk_description)/urdf/materials.xacro" />
     <!-- import empty link -->
+    <link name="base_link"/>
+    <!-- uncomment this part to fixed the body in space (ignore gravity)
     <link name="world"/>
-    <link name="base_link"/>
     <joint name="world2base" type="fixed">
         <origin xyz="0 0 0" rpy="0 0 0" />
@@ -13,4 +14,5 @@
         <child link="base_link"/>
     </joint>
+    -->
     <!-- Import robot parts -->
     <xacro:include filename="$(find gk_description)/urdf/body/body.urdf.xacro"/>
