Commit message: clean up version1 files

File: opr_description/urdf/version1/arms/left_arm.urdf.xacro (robot description, xacro)
@@ -33,5 +33,5 @@
             <origin xyz="0 0 0" rpy="0 0 0"/>
             <geometry>
-                <mesh filename="package://opr_description/meshes/STL/ARMS/body_to_arm.stl" />
+                <mesh filename="package://opr_description/meshes/version1/STL/ARMS/body_to_arm.stl" />
             </geometry>
             <material name="grey" />
@@ -40,5 +40,5 @@
             <origin xyz="0 0 0" rpy="0 0 0"/>
             <geometry>
-                <mesh filename="package://opr_description/meshes/STL/ARMS/body_to_arm.stl" />
+                <mesh filename="package://opr_description/meshes/version1/STL/ARMS/body_to_arm.stl" />
             </geometry>
         </collision>
@@ -53,5 +53,5 @@
             <origin xyz="0 0 -0.042" rpy="0 0 ${PI}"/>
             <geometry>
-                <mesh filename="package://opr_description/meshes/STL/ARMS/left_arm.stl" />
+                <mesh filename="package://opr_description/meshes/version1/STL/ARMS/left_arm.stl" />
             </geometry>
             <material name="blue" />
@@ -60,5 +60,5 @@
             <origin xyz="0 0 -0.042" rpy="0 0 ${PI}"/>
             <geometry>
-                <mesh filename="package://opr_description/meshes/STL/ARMS/left_arm.stl" />
+                <mesh filename="package://opr_description/meshes/version1/STL/ARMS/left_arm.stl" />
             </geometry>
         </collision>
@@ -73,5 +73,5 @@
             <origin xyz="0.09 0 0" rpy="0 0 0"/>
             <geometry>
-                <mesh filename="package://opr_description/meshes/STL/ARMS/hand.stl" />
+                <mesh filename="package://opr_description/meshes/version1/STL/ARMS/hand.stl" />
             </geometry>
             <material name="black" />
@@ -80,5 +80,5 @@
             <origin xyz="0.09 0 0" rpy="0 0 0"/>
             <geometry>
-                <mesh filename="package://opr_description/meshes/STL/ARMS/hand.stl" />
+                <mesh filename="package://opr_description/meshes/version1/STL/ARMS/hand.stl" />
             </geometry>
         </collision>

File: opr_description/urdf/version1/arms/right_arm.urdf.xacro (robot description, xacro)
@@ -33,5 +33,5 @@
             <origin xyz="0 0 0" rpy="0 0 ${PI}"/>
             <geometry>
-                <mesh filename="package://opr_description/meshes/STL/ARMS/body_to_arm.stl" />
+                <mesh filename="package://opr_description/meshes/version1/STL/ARMS/body_to_arm.stl" />
             </geometry>
             <material name="grey" />
@@ -40,5 +40,5 @@
             <origin xyz="0 0 0" rpy="0 0 ${PI}"/>
             <geometry>
-                <mesh filename="package://opr_description/meshes/STL/ARMS/body_to_arm.stl" />
+                <mesh filename="package://opr_description/meshes/version1/STL/ARMS/body_to_arm.stl" />
             </geometry>
         </collision>
@@ -53,5 +53,5 @@
             <origin xyz="0 0 -0.042" rpy="0 0 ${PI}"/>
             <geometry>
-                <mesh filename="package://opr_description/meshes/STL/ARMS/right_arm.stl" />
+                <mesh filename="package://opr_description/meshes/version1/STL/ARMS/right_arm.stl" />
             </geometry>
             <material name="blue" />
@@ -60,5 +60,5 @@
             <origin xyz="0 0 -0.042" rpy="0 0 ${PI}"/>
             <geometry>
-                <mesh filename="package://opr_description/meshes/STL/ARMS/right_arm.stl" />
+                <mesh filename="package://opr_description/meshes/version1/STL/ARMS/right_arm.stl" />
             </geometry>
         </collision>
@@ -73,5 +73,5 @@
             <origin xyz="0.09 0 0" rpy="${PI} 0 0"/>
             <geometry>
-                <mesh filename="package://opr_description/meshes/STL/ARMS/hand.stl" />
+                <mesh filename="package://opr_description/meshes/version1/STL/ARMS/hand.stl" />
             </geometry>
             <material name="black" />
@@ -80,5 +80,5 @@
             <origin xyz="0.09 0 0" rpy="${PI} 0 0"/>
             <geometry>
-                <mesh filename="package://opr_description/meshes/STL/ARMS/hand.stl" />
+                <mesh filename="package://opr_description/meshes/version1/STL/ARMS/hand.stl" />
             </geometry>
         </collision>

File: opr_description/urdf/version1/body/body.urdf.xacro (robot description, xacro)
@@ -17,5 +17,5 @@
             <origin xyz="0.005 0 0" rpy="0 0 ${PI/2}"/>
             <geometry>
-                <mesh filename="package://opr_description/meshes/STL/BODY/body.stl" />
+                <mesh filename="package://opr_description/meshes/version1/STL/BODY/body.stl" />
             </geometry>
             <material name="white" />
@@ -24,5 +24,5 @@
             <origin xyz="0.005 0 0" rpy="0 0 ${PI/2}"/>
             <geometry>
-                <mesh filename="package://opr_description/meshes/STL/BODY/body.stl" />
+                <mesh filename="package://opr_description/meshes/version1/STL/BODY/body.stl" />
             </geometry>
         </collision>

File: opr_description/urdf/version1/head/head.urdf.xacro (robot description, xacro)
@@ -26,5 +26,5 @@
             <origin xyz="0 0 0" rpy="0 0 0"/>
             <geometry>
-                <mesh filename="package://opr_description/meshes/STL/HEAD/head_yaw.stl" />
+                <mesh filename="package://opr_description/meshes/version1/STL/HEAD/head_yaw.stl" />
             </geometry>
             <material name="grey" />
@@ -33,5 +33,5 @@
             <origin xyz="0 0 0" rpy="0 0 0"/>
             <geometry>
-                <mesh filename="package://opr_description/meshes/STL/HEAD/head_yaw.stl" />
+                <mesh filename="package://opr_description/meshes/version1/STL/HEAD/head_yaw.stl" />
             </geometry>
         </collision>
@@ -46,5 +46,5 @@
             <origin xyz="0.0235 0 0.006" rpy="0 0 0"/>
             <geometry>
-                <mesh filename="package://opr_description/meshes/STL/HEAD/head_pitch.stl" />
+                <mesh filename="package://opr_description/meshes/version1/STL/HEAD/head_pitch.stl" />
             </geometry>
             <material name="white" />
@@ -53,5 +53,5 @@
             <origin xyz="0.0235 0 0.006" rpy="0 0 0"/>
             <geometry>
-                <mesh filename="package://opr_description/meshes/STL/HEAD/head_pitch.stl" />
+                <mesh filename="package://opr_description/meshes/version1/STL/HEAD/head_pitch.stl" />
             </geometry>
         </collision>

File: opr_description/urdf/version1/legs/left_leg.urdf.xacro (robot description, xacro)
@@ -2,74 +2,74 @@
 <robot xmlns:xacro="http://www.ros.org/wiki/xacro">
     <!-- leg joints -->
-    <joint name="right_waist_yaw_joint" type="revolute" >
+    <joint name="left_waist_yaw_joint" type="revolute" >
         <parent link="body_link" />
-        <child link="right_waist_yaw_link" />
-        <origin xyz="0.005 -0.044 -0.0575" rpy="0 0 0" />
+        <child link="left_waist_yaw_link" />
+        <origin xyz="0.005 0.044 -0.0575" rpy="0 0 0" />
         <limit effort="1000" lower="${-3*PI/4}" upper="${3*PI/4}" velocity="1.0" />
         <axis xyz="0 0 1" />
     </joint>
-    <joint name="right_waist_roll_joint" type="revolute" >
-        <parent link="right_waist_yaw_link" />
-        <child link="right_waist_roll_link" />
+    <joint name="left_waist_roll_joint" type="revolute" >
+        <parent link="left_waist_yaw_link" />
+        <child link="left_waist_roll_link" />
         <origin xyz="-0.0035 0 -0.0389" rpy="0 0 0" />
         <limit effort="1000" lower="${-PI/2}" upper="${PI/2}" velocity="1.0" />
         <axis xyz="1 0 0" />
     </joint>
-    <joint name="right_waist_front_pitch_joint" type="revolute" >
-        <parent link="right_waist_roll_link" />
-        <child link="right_waist_front_pitch_link" />
+    <joint name="left_waist_front_pitch_joint" type="revolute" >
+        <parent link="left_waist_roll_link" />
+        <child link="left_waist_front_pitch_link" />
         <origin xyz="0.0121 0 0.00062" rpy="0 0 0" />
-        <mimic joint="right_waist_pitch_joint" multiplier="-1" offset="0" />
+        <mimic joint="left_waist_pitch_joint" multiplier="-1" offset="0" />
         <limit effort="1000" lower="${-PI/2}" upper="${PI/6}" velocity="1.0" />
         <axis xyz="0 1 0" />
     </joint>
-    <joint name="right_waist_back_pitch_joint" type="revolute" >
-        <parent link="right_waist_roll_link" />
-        <child link="right_waist_back_pitch_link" />
+    <joint name="left_waist_back_pitch_joint" type="revolute" >
+        <parent link="left_waist_roll_link" />
+        <child link="left_waist_back_pitch_link" />
         <origin xyz="-0.0198 0 -0.0194" rpy="0 0 0" />
-        <mimic joint="right_waist_pitch_joint" multiplier="-1" offset="0" />
+        <mimic joint="left_waist_pitch_joint" multiplier="-1" offset="0" />
         <limit effort="1000" lower="${-PI/2}" upper="${PI/6}" velocity="1.0" />
         <axis xyz="0 1 0" />
     </joint>
-    <joint name="right_waist_pitch_joint" type="revolute" >
-        <parent link="right_waist_back_pitch_link" />
-        <child link="right_knee_pitch_link" />
+    <joint name="left_waist_pitch_joint" type="revolute" >
+        <parent link="left_waist_back_pitch_link" />
+        <child link="left_knee_pitch_link" />
         <origin xyz="0 0 -0.1" rpy="0 0 0" />
         <limit effort="1000" lower="${-PI/6}" upper="${PI/2}" velocity="1.0" />
         <axis xyz="0 1 0" />
     </joint>
-    <joint name="right_knee_pitch_joint" type="revolute" >
-        <parent link="right_knee_pitch_link" />
-        <child link="right_shin_back_pitch_link" />
+    <joint name="left_knee_pitch_joint" type="revolute" >
+        <parent link="left_knee_pitch_link" />
+        <child link="left_shin_back_pitch_link" />
         <origin xyz="0 0 -0.017" rpy="0 0 0" />
         <limit effort="1000" lower="${-PI/6}" upper="${PI/2}" velocity="1.0" />
         <axis xyz="0 1 0" />
     </joint>
-    <joint name="right_knee_front_pitch_joint" type="revolute" >
-        <parent link="right_knee_pitch_link" />
-        <child link="right_shin_front_pitch_link" />
+    <joint name="left_knee_front_pitch_joint" type="revolute" >
+        <parent link="left_knee_pitch_link" />
+        <child link="left_shin_front_pitch_link" />
         <origin xyz="0.0319 0 -0.037" rpy="0 0 0" />
-        <mimic joint="right_knee_pitch_joint" multiplier="1" offset="0" />
-        <limit effort="1000" lower="${-PI/6}" upper="${PI/2}" velocity="1.0" />
-        <axis xyz="0 1 0" />
-    </joint>
-    <joint name="right_ankle_independent_pitch_joint" type="revolute" >
-        <parent link="right_shin_front_pitch_link" />
-        <child link="right_independent_pitch_link" />
+        <mimic joint="left_knee_pitch_joint" multiplier="1" offset="0" />
+        <limit effort="1000" lower="${-PI/6}" upper="${PI/2}" velocity="1.0" />
+        <axis xyz="0 1 0" />
+    </joint>
+    <joint name="left_ankle_independent_pitch_joint" type="revolute" >
+        <parent link="left_shin_front_pitch_link" />
+        <child link="left_independent_pitch_link" />
         <origin xyz="0 0 -0.1" rpy="0 0 0" />
-        <mimic joint="right_knee_pitch_joint" multiplier="-1" offset="0" />
-        <limit effort="1000" lower="${-PI/6}" upper="${PI/2}" velocity="1.0" />
-        <axis xyz="0 1 0" />
-    </joint>
-    <joint name="right_ankle_pitch_joint" type="revolute" >
-        <parent link="right_independent_pitch_link" />
-        <child link="right_ankle_pitch_link" />
+        <mimic joint="left_knee_pitch_joint" multiplier="-1" offset="0" />
+        <limit effort="1000" lower="${-PI/6}" upper="${PI/2}" velocity="1.0" />
+        <axis xyz="0 1 0" />
+    </joint>
+    <joint name="left_ankle_pitch_joint" type="revolute" >
+        <parent link="left_independent_pitch_link" />
+        <child link="left_ankle_pitch_link" />
         <origin xyz="0 0 0" rpy="0 0 0" />
         <limit effort="1000" lower="${-3*PI/4}" upper="${3*PI/4}" velocity="1.0" />
         <axis xyz="0 1 0" />
     </joint>
-    <joint name="right_ankle_roll_joint" type="revolute" >
-        <parent link="right_ankle_pitch_link" />
-        <child link="right_foot_link" />
+    <joint name="left_ankle_roll_joint" type="revolute" >
+        <parent link="left_ankle_pitch_link" />
+        <child link="left_foot_link" />
         <origin xyz="-0.0325 0 0" rpy="0 0 0"/>
         <limit effort="1000" lower="${-PI/2}" upper="${PI/2}" velocity="1.0" />
@@ -77,5 +77,5 @@
     </joint>
     <!-- leg links -->
-    <link name="right_waist_yaw_link">
+    <link name="left_waist_yaw_link">
         <inertial>
             <mass value="1.0"/>
@@ -86,5 +86,5 @@
             <origin xyz="0 0 0" rpy="0 0 ${PI/2}"/>
             <geometry>
-                <mesh filename="package://opr_description/meshes/STL/LEGS/body_to_waist.stl" />
+                <mesh filename="package://opr_description/meshes/version1/STL/LEGS/body_to_waist.stl" />
             </geometry>
             <material name="grey" />
@@ -93,9 +93,9 @@
             <origin xyz="0 0 0" rpy="0 0 ${PI/2}"/>
             <geometry>
-                <mesh filename="package://opr_description/meshes/STL/LEGS/body_to_waist.stl" />
-            </geometry>
-        </collision>
-    </link>
-    <link name="right_waist_roll_link">
+                <mesh filename="package://opr_description/meshes/version1/STL/LEGS/body_to_waist.stl" />
+            </geometry>
+        </collision>
+    </link>
+    <link name="left_waist_roll_link">
         <inertial>
             <mass value="1.0"/>
@@ -106,5 +106,5 @@
             <origin xyz="0 0 0.003" rpy="0 0 0"/>
             <geometry>
-                <mesh filename="package://opr_description/meshes/STL/LEGS/waist.stl" />
+                <mesh filename="package://opr_description/meshes/version1/STL/LEGS/waist.stl" />
             </geometry>
             <material name="white" />
@@ -113,9 +113,9 @@
             <origin xyz="0 0 0.003" rpy="0 0 0"/>
             <geometry>
-                <mesh filename="package://opr_description/meshes/STL/LEGS/waist.stl" />
-            </geometry>
-        </collision>
-    </link>
-    <link name="right_waist_front_pitch_link">
+                <mesh filename="package://opr_description/meshes/version1/STL/LEGS/waist.stl" />
+            </geometry>
+        </collision>
+    </link>
+    <link name="left_waist_front_pitch_link">
         <inertial>
             <mass value="1.0"/>
@@ -126,5 +126,5 @@
             <origin xyz="-0.001 0 -0.05" rpy="0 0 0"/>
             <geometry>
-                <mesh filename="package://opr_description/meshes/STL/LEGS/front_link.stl" />
+                <mesh filename="package://opr_description/meshes/version1/STL/LEGS/front_link.stl" />
             </geometry>
             <material name="blue" />
@@ -133,9 +133,9 @@
             <origin xyz="-0.001 0 -0.05" rpy="0 0 0"/>
             <geometry>
-                <mesh filename="package://opr_description/meshes/STL/LEGS/front_link.stl" />
-            </geometry>
-        </collision>
-    </link>
-    <link name="right_waist_back_pitch_link">
+                <mesh filename="package://opr_description/meshes/version1/STL/LEGS/front_link.stl" />
+            </geometry>
+        </collision>
+    </link>
+    <link name="left_waist_back_pitch_link">
         <inertial>
             <mass value="1.0"/>
@@ -146,5 +146,5 @@
             <origin xyz="0.001 0 -0.05" rpy="${PI} 0 ${PI}"/>
             <geometry>
-                <mesh filename="package://opr_description/meshes/STL/LEGS/back_link.stl" />
+                <mesh filename="package://opr_description/meshes/version1/STL/LEGS/back_link.stl" />
             </geometry>
             <material name="blue" />
@@ -153,9 +153,9 @@
             <origin xyz="0.001 0 -0.05" rpy="${PI} 0 ${PI}"/>
             <geometry>
-                <mesh filename="package://opr_description/meshes/STL/LEGS/back_link.stl" />
-            </geometry>
-        </collision>
-    </link>
-    <link name="right_knee_pitch_link">
+                <mesh filename="package://opr_description/meshes/version1/STL/LEGS/back_link.stl" />
+            </geometry>
+        </collision>
+    </link>
+    <link name="left_knee_pitch_link">
         <inertial>
             <mass value="1.0"/>
@@ -166,5 +166,5 @@
             <origin xyz="0.0002 0 0.0002" rpy="0 0 0"/>
             <geometry>
-                <mesh filename="package://opr_description/meshes/STL/LEGS/right_knee.stl" />
+                <mesh filename="package://opr_description/meshes/version1/STL/LEGS/left_knee.stl" />
             </geometry>
             <material name="white" />
@@ -173,9 +173,9 @@
             <origin xyz="0.0002 0 0.0002" rpy="0 0 0"/>
             <geometry>
-                <mesh filename="package://opr_description/meshes/STL/LEGS/right_knee.stl" />
-            </geometry>
-        </collision>
-    </link>
-    <link name="right_shin_front_pitch_link">
+                <mesh filename="package://opr_description/meshes/version1/STL/LEGS/left_knee.stl" />
+            </geometry>
+        </collision>
+    </link>
+    <link name="left_shin_front_pitch_link">
         <inertial>
             <mass value="1.0"/>
@@ -186,5 +186,5 @@
             <origin xyz="-0.001 0 -0.05" rpy="${PI} 0 0"/>
             <geometry>
-                <mesh filename="package://opr_description/meshes/STL/LEGS/front_link.stl" />
+                <mesh filename="package://opr_description/meshes/version1/STL/LEGS/front_link.stl" />
             </geometry>
             <material name="blue" />
@@ -193,9 +193,9 @@
             <origin xyz="-0.001 0 -0.05" rpy="${PI} 0 0"/>
             <geometry>
-                <mesh filename="package://opr_description/meshes/STL/LEGS/front_link.stl" />
-            </geometry>
-        </collision>
-    </link>
-    <link name="right_shin_back_pitch_link">
+                <mesh filename="package://opr_description/meshes/version1/STL/LEGS/front_link.stl" />
+            </geometry>
+        </collision>
+    </link>
+    <link name="left_shin_back_pitch_link">
         <inertial>
             <mass value="1.0"/>
@@ -206,5 +206,5 @@
             <origin xyz="0.001 0 -0.05" rpy="0 0 ${PI}"/>
             <geometry>
-                <mesh filename="package://opr_description/meshes/STL/LEGS/back_link.stl" />
+                <mesh filename="package://opr_description/meshes/version1/STL/LEGS/back_link.stl" />
             </geometry>
             <material name="blue" />
@@ -213,9 +213,9 @@
             <origin xyz="0.001 0 -0.05" rpy="0 0 ${PI}"/>
             <geometry>
-                <mesh filename="package://opr_description/meshes/STL/LEGS/back_link.stl" />
-            </geometry>
-        </collision>
-    </link>
-    <link name="right_independent_pitch_link">
+                <mesh filename="package://opr_description/meshes/version1/STL/LEGS/back_link.stl" />
+            </geometry>
+        </collision>
+    </link>
+    <link name="left_independent_pitch_link">
         <inertial>
             <mass value="1.0"/>
@@ -226,5 +226,5 @@
             <origin xyz="0 0 0" rpy="${PI/2} ${PI/7} ${PI}"/>
             <geometry>
-                <mesh filename="package://opr_description/meshes/STL/LEGS/ankle_pitch.stl" />
+                <mesh filename="package://opr_description/meshes/version1/STL/LEGS/ankle_pitch.stl" />
             </geometry>
             <material name="grey" />
@@ -233,9 +233,9 @@
             <origin xyz="0 0 0" rpy="${PI/2} ${PI/7} ${PI}"/>
             <geometry>
-                <mesh filename="package://opr_description/meshes/STL/LEGS/ankle_pitch.stl" />
-            </geometry>
-        </collision>
-    </link>
-    <link name="right_ankle_pitch_link">
+                <mesh filename="package://opr_description/meshes/version1/STL/LEGS/ankle_pitch.stl" />
+            </geometry>
+        </collision>
+    </link>
+    <link name="left_ankle_pitch_link">
         <inertial>
             <mass value="1.0"/>
@@ -246,5 +246,5 @@
             <origin xyz="-0.0137 0 0" rpy="0 0 0"/>
             <geometry>
-                <mesh filename="package://opr_description/meshes/STL/LEGS/right_ankle.stl" />
+                <mesh filename="package://opr_description/meshes/version1/STL/LEGS/left_ankle.stl" />
             </geometry>
             <material name="white" />
@@ -253,9 +253,9 @@
             <origin xyz="-0.0137 0 0" rpy="0 0 0"/>
             <geometry>
-                <mesh filename="package://opr_description/meshes/STL/LEGS/right_ankle.stl" />
-            </geometry>
-        </collision>
-    </link>
-    <link name="right_foot_link">
+                <mesh filename="package://opr_description/meshes/version1/STL/LEGS/left_ankle.stl" />
+            </geometry>
+        </collision>
+    </link>
+    <link name="left_foot_link">
         <inertial>
             <mass value="1.0"/>
@@ -266,5 +266,5 @@
             <origin xyz="0 0 0" rpy="0 0 0"/>
             <geometry>
-                <mesh filename="package://opr_description/meshes/STL/LEGS/right_foot.stl" />
+                <mesh filename="package://opr_description/meshes/version1/STL/LEGS/left_foot.stl" />
             </geometry>
             <material name="black" />
@@ -273,5 +273,5 @@
             <origin xyz="0 0 0" rpy="0 0 0"/>
             <geometry>
-                <mesh filename="package://opr_description/meshes/STL/LEGS/right_foot.stl" />
+                <mesh filename="package://opr_description/meshes/version1/STL/LEGS/left_foot.stl" />
             </geometry>
         </collision>
