Commit message: fix indent

File: opr_description/urdf/version1/arms/left_arm.urdf.xacro (robot description, xacro)
@@ -29,5 +29,5 @@
             <origin xyz="0 0 0"/>
             <inertia ixx="1.0" ixy="0.0" ixz="0.0" iyy="1.0" iyz="0.0" izz="1.0"/>
-            </inertial>
+        </inertial>
         <visual>
             <origin xyz="0 0 0" rpy="0 0 0"/>
@@ -49,5 +49,5 @@
             <origin xyz="0 0 0"/>
             <inertia ixx="1.0" ixy="0.0" ixz="0.0" iyy="1.0" iyz="0.0" izz="1.0"/>
-            </inertial>
+        </inertial>
         <visual>
             <origin xyz="0 0 -0.042" rpy="0 0 ${PI}"/>
@@ -69,5 +69,5 @@
             <origin xyz="0 0 0"/>
             <inertia ixx="1.0" ixy="0.0" ixz="0.0" iyy="1.0" iyz="0.0" izz="1.0"/>
-            </inertial>
+        </inertial>
         <visual>
             <origin xyz="0.09 0 0" rpy="0 0 0"/>

File: opr_description/urdf/version1/arms/right_arm.urdf.xacro (robot description, xacro)
@@ -29,5 +29,5 @@
             <origin xyz="0 0 0"/>
             <inertia ixx="1.0" ixy="0.0" ixz="0.0" iyy="1.0" iyz="0.0" izz="1.0"/>
-            </inertial>
+        </inertial>
         <visual>
             <origin xyz="0 0 0" rpy="0 0 ${PI}"/>
@@ -49,5 +49,5 @@
             <origin xyz="0 0 0"/>
             <inertia ixx="1.0" ixy="0.0" ixz="0.0" iyy="1.0" iyz="0.0" izz="1.0"/>
-            </inertial>
+        </inertial>
         <visual>
             <origin xyz="0 0 -0.042" rpy="0 0 ${PI}"/>
@@ -69,5 +69,5 @@
             <origin xyz="0 0 0"/>
             <inertia ixx="1.0" ixy="0.0" ixz="0.0" iyy="1.0" iyz="0.0" izz="1.0"/>
-            </inertial>
+        </inertial>
         <visual>
             <origin xyz="0.09 0 0" rpy="${PI} 0 0"/>

File: opr_description/urdf/version1/body/body.urdf.xacro (robot description, xacro)
@@ -13,5 +13,5 @@
             <origin xyz="0 0 0"/>
             <inertia ixx="1.0" ixy="0.0" ixz="0.0" iyy="1.0" iyz="0.0" izz="1.0"/>
-            </inertial>
+        </inertial>
         <visual>
             <origin xyz="0.005 0 0" rpy="0 0 ${PI/2}"/>

File: opr_description/urdf/version1/head/head.urdf.xacro (robot description, xacro)
@@ -22,5 +22,5 @@
             <origin xyz="0 0 0"/>
             <inertia ixx="1.0" ixy="0.0" ixz="0.0" iyy="1.0" iyz="0.0" izz="1.0"/>
-            </inertial>
+        </inertial>
         <visual>
             <origin xyz="0 0 0" rpy="0 0 0"/>
@@ -42,5 +42,5 @@
             <origin xyz="0 0 0"/>
             <inertia ixx="1.0" ixy="0.0" ixz="0.0" iyy="1.0" iyz="0.0" izz="1.0"/>
-            </inertial>
+        </inertial>
         <visual>
             <origin xyz="0.0235 0 0.006" rpy="0 0 0"/>

File: opr_description/urdf/version1/legs/left_leg.urdf.xacro (robot description, xacro)
@@ -82,5 +82,5 @@
             <origin xyz="0 0 0"/>
             <inertia ixx="1.0" ixy="0.0" ixz="0.0" iyy="1.0" iyz="0.0" izz="1.0"/>
-            </inertial>
+        </inertial>
         <visual>
             <origin xyz="0 0 0" rpy="0 0 ${PI/2}"/>
@@ -102,5 +102,5 @@
             <origin xyz="0 0 0"/>
             <inertia ixx="1.0" ixy="0.0" ixz="0.0" iyy="1.0" iyz="0.0" izz="1.0"/>
-            </inertial>
+        </inertial>
         <visual>
             <origin xyz="0 0 0.003" rpy="0 0 0"/>
@@ -122,5 +122,5 @@
             <origin xyz="0 0 0"/>
             <inertia ixx="1.0" ixy="0.0" ixz="0.0" iyy="1.0" iyz="0.0" izz="1.0"/>
-            </inertial>
+        </inertial>
         <visual>
             <origin xyz="-0.001 0 -0.05" rpy="0 0 0"/>
@@ -142,5 +142,5 @@
             <origin xyz="0 0 0"/>
             <inertia ixx="1.0" ixy="0.0" ixz="0.0" iyy="1.0" iyz="0.0" izz="1.0"/>
-            </inertial>
+        </inertial>
         <visual>
             <origin xyz="0.001 0 -0.05" rpy="${PI} 0 ${PI}"/>
@@ -162,5 +162,5 @@
             <origin xyz="0 0 0"/>
             <inertia ixx="1.0" ixy="0.0" ixz="0.0" iyy="1.0" iyz="0.0" izz="1.0"/>
-            </inertial>
+        </inertial>
         <visual>
             <origin xyz="0.0002 0 0.0002" rpy="0 0 0"/>
@@ -182,5 +182,5 @@
             <origin xyz="0 0 0"/>
             <inertia ixx="1.0" ixy="0.0" ixz="0.0" iyy="1.0" iyz="0.0" izz="1.0"/>
-            </inertial>
+        </inertial>
         <visual>
             <origin xyz="-0.001 0 -0.05" rpy="${PI} 0 0"/>
@@ -202,5 +202,5 @@
             <origin xyz="0 0 0"/>
             <inertia ixx="1.0" ixy="0.0" ixz="0.0" iyy="1.0" iyz="0.0" izz="1.0"/>
-            </inertial>
+        </inertial>
         <visual>
             <origin xyz="0.001 0 -0.05" rpy="0 0 ${PI}"/>
@@ -222,5 +222,5 @@
             <origin xyz="0 0 0"/>
             <inertia ixx="1.0" ixy="0.0" ixz="0.0" iyy="1.0" iyz="0.0" izz="1.0"/>
-            </inertial>
+        </inertial>
         <visual>
             <origin xyz="0 0 0" rpy="${PI/2} ${PI/7} ${PI}"/>
@@ -242,5 +242,5 @@
             <origin xyz="0 0 0"/>
             <inertia ixx="1.0" ixy="0.0" ixz="0.0" iyy="1.0" iyz="0.0" izz="1.0"/>
-            </inertial>
+        </inertial>
         <visual>
             <origin xyz="-0.0137 0 0" rpy="0 0 0"/>
@@ -262,5 +262,5 @@
             <origin xyz="0 0 0"/>
             <inertia ixx="1.0" ixy="0.0" ixz="0.0" iyy="1.0" iyz="0.0" izz="1.0"/>
-            </inertial>
+        </inertial>
         <visual>
             <origin xyz="0 0 0" rpy="0 0 0"/>

File: opr_description/urdf/version1/legs/right_leg.urdf.xacro (robot description, xacro)
@@ -82,5 +82,5 @@
             <origin xyz="0 0 0"/>
             <inertia ixx="1.0" ixy="0.0" ixz="0.0" iyy="1.0" iyz="0.0" izz="1.0"/>
-            </inertial>
+        </inertial>
         <visual>
             <origin xyz="0 0 0" rpy="0 0 ${PI/2}"/>
@@ -102,5 +102,5 @@
             <origin xyz="0 0 0"/>
             <inertia ixx="1.0" ixy="0.0" ixz="0.0" iyy="1.0" iyz="0.0" izz="1.0"/>
-            </inertial>
+        </inertial>
         <visual>
             <origin xyz="0 0 0.003" rpy="0 0 0"/>
@@ -122,5 +122,5 @@
             <origin xyz="0 0 0"/>
             <inertia ixx="1.0" ixy="0.0" ixz="0.0" iyy="1.0" iyz="0.0" izz="1.0"/>
-            </inertial>
+        </inertial>
         <visual>
             <origin xyz="-0.001 0 -0.05" rpy="0 0 0"/>
@@ -142,5 +142,5 @@
             <origin xyz="0 0 0"/>
             <inertia ixx="1.0" ixy="0.0" ixz="0.0" iyy="1.0" iyz="0.0" izz="1.0"/>
-            </inertial>
+        </inertial>
         <visual>
             <origin xyz="0.001 0 -0.05" rpy="${PI} 0 ${PI}"/>
@@ -162,5 +162,5 @@
             <origin xyz="0 0 0"/>
             <inertia ixx="1.0" ixy="0.0" ixz="0.0" iyy="1.0" iyz="0.0" izz="1.0"/>
-            </inertial>
+        </inertial>
         <visual>
             <origin xyz="0.0002 0 0.0002" rpy="0 0 0"/>
@@ -182,5 +182,5 @@
             <origin xyz="0 0 0"/>
             <inertia ixx="1.0" ixy="0.0" ixz="0.0" iyy="1.0" iyz="0.0" izz="1.0"/>
-            </inertial>
+        </inertial>
         <visual>
             <origin xyz="-0.001 0 -0.05" rpy="${PI} 0 0"/>
@@ -202,5 +202,5 @@
             <origin xyz="0 0 0"/>
             <inertia ixx="1.0" ixy="0.0" ixz="0.0" iyy="1.0" iyz="0.0" izz="1.0"/>
-            </inertial>
+        </inertial>
         <visual>
             <origin xyz="0.001 0 -0.05" rpy="0 0 ${PI}"/>
@@ -222,5 +222,5 @@
             <origin xyz="0 0 0"/>
             <inertia ixx="1.0" ixy="0.0" ixz="0.0" iyy="1.0" iyz="0.0" izz="1.0"/>
-            </inertial>
+        </inertial>
         <visual>
             <origin xyz="0 0 0" rpy="${PI/2} ${PI/7} ${PI}"/>
@@ -242,5 +242,5 @@
             <origin xyz="0 0 0"/>
             <inertia ixx="1.0" ixy="0.0" ixz="0.0" iyy="1.0" iyz="0.0" izz="1.0"/>
-            </inertial>
+        </inertial>
         <visual>
             <origin xyz="-0.0137 0 0" rpy="0 0 0"/>
@@ -262,5 +262,5 @@
             <origin xyz="0 0 0"/>
             <inertia ixx="1.0" ixy="0.0" ixz="0.0" iyy="1.0" iyz="0.0" izz="1.0"/>
-            </inertial>
+        </inertial>
         <visual>
             <origin xyz="0 0 0" rpy="0 0 0"/>
